File: kicad/kicad.kicad_pcb (KiCad board)
At the start: 2 copper layers, 121 parts, among them Q1 PMF170XP,115, Q2 FS8205A_C2830320, SW1 TS-1088-AR02016, U1 74AHC1G14GW,125, U2 E73-2G4M08S1C, U3 BL8573CS8TR, U4 DW01A, U5 S2B-PH-K-S(LF)(SN), U6 LP5024RSMR, U7 SN74HCS74BQAR, X1 FC-13532.768KHZ9PF20PPM, X2 XTM20032000DT00351005

Commit message: changed raw mcu to e73module with antena... cleaned pcb a little
Parts:
- removed C1, C2, C6, C9: GRM188C71C475KE21D, easyeda2kicad:C0603
- removed C10, C8: GRM155C71C105KE11D, easyeda2kicad:C0402
- removed C12, C15, C16, C7: GRM033C71C104KE14D, easyeda2kicad:C0201
- removed C13: CL05B473KO5NNNC, easyeda2kicad:C0402
- removed C14, C21: N.C., easyeda2kicad:C0402
- removed C17, C18, C4, C5: 0402CG120F500NT, easyeda2kicad:C0402
- removed C19: GJM1555C1HR80WB01D, easyeda2kicad:C0402
- removed C20: GRM1555C1H821FA01D, easyeda2kicad:C0402
- removed C22: GJM1555C1HR50WB01D, easyeda2kicad:C0402
- removed C23: N.C, easyeda2kicad:C0402
- removed C24: GCM1555C1H101FA16D, easyeda2kicad:C0402
- removed L3: 0402DC-4N7XJRW, easyeda2kicad:IND-SMD_L1.1-W0.6
- removed L4: BRC2016T100K, easyeda2kicad:IND-SMD_L2.0-W1.6_BRC2016
- removed NRF1: NRF52840-QIAA-R7, Package_DFN_QFN:Nordic_AQFN-73-1EP_7x7mm_P0.5mm
- removed X1: FC-13532.768KHZ9PF20PPM, easyeda2kicad:OSC-SMD_L3.2-W1.5
- removed X2: XTM20032000DT00351005, easyeda2kicad:CRYSTAL-SMD_4P-L2.0-W1.6-BL-A
- added C27: GRM188C71C475KE21D, easyeda2kicad:C0603, F.Cu at (197.8, 101.0)
- added C28: 0402CG120F500NT, easyeda2kicad:C0402, F.Cu at (189.3, 84.7)
- added C29: 0402CG120F500NT, easyeda2kicad:C0402, F.Cu at (189.3, 88.8)
- added X3: FC-13532.768KHZ9PF20PPM, easyeda2kicad:OSC-SMD_L3.2-W1.5, F.Cu at (191.8, 86.8)
- moved SW1 112.5 mm to (192.0, 101.1)
- moved C11 98.5 mm to (193.1, 98.6)
- moved R12 97.6 mm to (211.7, 104.3)
- moved R13 97.0 mm to (209.5, 104.3)
- moved R14 96.5 mm to (207.3, 104.3)
- moved R6 96.5 mm to (181.4, 76.4)
- moved R7 96.5 mm to (181.4, 78.5)
- moved R5 95.4 mm to (191.2, 98.6)
- moved R11 89.6 mm to (217.5, 108.9)
- moved C25 87.2 mm to (221.7, 109.0)
- moved L1 84.3 mm to (191.8, 95.3), turned to 180 degrees
- moved U6 82.9 mm to (209.4, 107.6)
- moved F1 82.3 mm to (183.6, 70.6)
- moved U3 80.8 mm to (190.3, 55.5)
- moved D2 79.7 mm to (200.7, 65.5), turned to -90 degrees
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Connections:
- F1 pad 1: /VBUS -> Net-(F1-Pad1)
- F1 pad 2: Net-(U3-VCC) -> /VBUS
- L1 pad 1: /VDD_nRF -> Net-(U2-DCH)
- L1 pad 2: Net-(NRF1-DCCH) -> /VDD_nRF
- U2 pad 11: unconnected-(U2-XL1-Pad11) -> Net-(U2-XL1)
- U2 pad 13: unconnected-(U2-XL2-Pad13) -> Net-(U2-XL2)
- U2 pad 14: unconnected-(U2-P0.06-Pad14) -> /ROW2
- U2 pad 16: unconnected-(U2-P0.08-Pad16) -> /ROW3
- U2 pad 17: unconnected-(U2-P1.09-Pad17) -> /ROW4
- U2 pad 19: unconnected-(U2-VCC-Pad19) -> /VDD_nRF
- U2 pad 21: unconnected-(U2-GND-Pad21) -> GND
- U2 pad 23: unconnected-(U2-VDH-Pad23) -> /PWR
- U2 pad 24: unconnected-(U2-GND-Pad24) -> GND
- U2 pad 25: unconnected-(U2-DCH-Pad25) -> Net-(U2-DCH)
- U2 pad 26: unconnected-(U2-RST-Pad26) -> /RESET
- U2 pad 27: unconnected-(U2-VBS-Pad27) -> /VBUS
- U2 pad 29: unconnected-(U2-D--Pad29) -> /D-
- U2 pad 3: unconnected-(U2-P0.03-Pad3) -> /ROW1
- U2 pad 31: unconnected-(U2-D+-Pad31) -> /D+
- U2 pad 32: unconnected-(U2-P0.20-Pad32) -> /COL5
- U2 pad 33: unconnected-(U2-P0.13-Pad33) -> /COL4
- U2 pad 34: unconnected-(U2-P0.22-Pad34) -> /COL3
- U2 pad 35: unconnected-(U2-P0.24-Pad35) -> /COL2
- U2 pad 36: unconnected-(U2-P1.00-Pad36) -> /COL1
- U2 pad 37: unconnected-(U2-SWD-Pad37) -> /SWDIO
- U2 pad 39: unconnected-(U2-SWC-Pad39) -> /SWBCLK
- U2 pad 41: unconnected-(U2-NF1-Pad41) -> /LED_EN
- U2 pad 42: unconnected-(U2-P1.06-Pad42) -> /LED_SDA
- U2 pad 43: unconnected-(U2-NF2-Pad43) -> /LED_SCL
- U2 pad 5: unconnected-(U2-GND-Pad5) -> GND
- U2 pad 7: unconnected-(U2-AI0-Pad7) -> /ADC
- U2 pad 8: unconnected-(U2-AI5-Pad8) -> /CHRG
- U2 pad 9: unconnected-(U2-AI7-Pad9) -> /STDBY
- U3 pad 4: Net-(U3-VCC) -> /VBUS
- U6 pad 1: /LED0 -> /LED19
- U6 pad 10: /LED9 -> /LED8
- U6 pad 11: /LED10 -> /LED9
- U6 pad 12: /LED11 -> /LED10
- U6 pad 13: /LED12 -> /LED11
- U6 pad 14: /LED13 -> /LED12
- U6 pad 15: /LED14 -> /LED13
- U6 pad 16: /LED15 -> /LED14
- U6 pad 17: /LED16 -> /LED15
- U6 pad 18: /LED17 -> /LED16
- U6 pad 19: /LED18 -> /LED17
- U6 pad 2: /LED1 -> /LED0
- U6 pad 20: /LED19 -> /LED18
- U6 pad 3: /LED2 -> /LED1
- U6 pad 4: /LED3 -> /LED2
- U6 pad 5: /LED4 -> /LED3
- U6 pad 6: /LED5 -> /LED4
- U6 pad 7: /LED6 -> /LED5
- U6 pad 8: /LED7 -> /LED6
- U6 pad 9: /LED8 -> /LED7
- USBC1 pad A4B9: /VBUS -> Net-(F1-Pad1)
- USBC1 pad B4A9: /VBUS -> Net-(F1-Pad1)

Commit message: ...
Parts:
- removed REF**: 3500mAh LiPo, my:3500mAh LiPo
- added ?: , clipboard:b9cf7df6-7b49-4194-bf11-16aaca528749, F.Cu at (270.6, 24.1)
- added Battery?: 3500mAh LiPo, my:3500mAh LiPo, F.Cu at (129.5, 77.6)
- added hex_outline: , clipboard:b9cf7df6-7b49-4194-bf11-16aaca528749, F.Cu at (-69.4, 82.5)
- added hex_outline: , clipboard:b9cf7df6-7b49-4194-bf11-16aaca528749, F.Cu at (215.9, 49.4)
- added hex_outline: , clipboard:b9cf7df6-7b49-4194-bf11-16aaca528749, F.Cu at (104.2, 113.9)
- added hex_outline: , clipboard:b9cf7df6-7b49-4194-bf11-16aaca528749, F.Cu at (160.1, 81.7)
- added hex_outline: , clipboard:b9cf7df6-7b49-4194-bf11-16aaca528749, F.Cu at (178.7, 70.9)
- added hex_outline: , clipboard:b9cf7df6-7b49-4194-bf11-16aaca528749, F.Cu at (197.3, 81.7)
- added hex_outline: , clipboard:b9cf7df6-7b49-4194-bf11-16aaca528749, F.Cu at (122.8, 103.2)
- added hex_outline: , clipboard:b9cf7df6-7b49-4194-bf11-16aaca528749, F.Cu at (141.5, 49.4)
- added hex_outline: , clipboard:b9cf7df6-7b49-4194-bf11-16aaca528749, F.Cu at (-32.2, 61.0)
- added hex_outline: , clipboard:b9cf7df6-7b49-4194-bf11-16aaca528749, F.Cu at (-125.3, 28.8)
- added hex_outline: , clipboard:b9cf7df6-7b49-4194-bf11-16aaca528749, F.Cu at (-69.4, 61.0)
- added hex_outline: , clipboard:b9cf7df6-7b49-4194-bf11-16aaca528749, F.Cu at (-50.8, 7.30)
- added hex_outline: , clipboard:b9cf7df6-7b49-4194-bf11-16aaca528749, F.Cu at (-13.6, 50.3)
- added hex_outline: , clipboard:b9cf7df6-7b49-4194-bf11-16aaca528749, F.Cu at (-13.6, 71.8)
- added hex_outline: , clipboard:b9cf7df6-7b49-4194-bf11-16aaca528749, F.Cu at (-106.7, 82.5)
- added hex_outline: , clipboard:b9cf7df6-7b49-4194-bf11-16aaca528749, F.Cu at (122.8, 60.1)
- added hex_outline: , clipboard:b9cf7df6-7b49-4194-bf11-16aaca528749, F.Cu at (-69.4, 18.1)
- added hex_outline: , clipboard:b9cf7df6-7b49-4194-bf11-16aaca528749, F.Cu at (160.1, 38.6)
- added hex_outline: , clipboard:b9cf7df6-7b49-4194-bf11-16aaca528749, F.Cu at (-50.8, 50.3)
- added hex_outline: , clipboard:b9cf7df6-7b49-4194-bf11-16aaca528749, F.Cu at (-88.0, 93.3)
- added hex_outline: , clipboard:b9cf7df6-7b49-4194-bf11-16aaca528749, F.Cu at (-13.6, 28.8)
- added hex_outline: , clipboard:b9cf7df6-7b49-4194-bf11-16aaca528749, F.Cu at (-125.3, 93.3)
- added hex_outline: , clipboard:b9cf7df6-7b49-4194-bf11-16aaca528749, F.Cu at (160.1, 103.2)
- added hex_outline: , clipboard:b9cf7df6-7b49-4194-bf11-16aaca528749, F.Cu at (-125.3, 71.8)
- added hex_outline: , clipboard:b9cf7df6-7b49-4194-bf11-16aaca528749, F.Cu at (197.3, 38.6)
- added hex_outline: , clipboard:b9cf7df6-7b49-4194-bf11-16aaca528749, F.Cu at (215.9, 70.9)
- added hex_outline: , clipboard:b9cf7df6-7b49-4194-bf11-16aaca528749, F.Cu at (104.2, 92.4)
- added hex_outline: , clipboard:b9cf7df6-7b49-4194-bf11-16aaca528749, F.Cu at (215.9, 92.4)
- added hex_outline: , clipboard:b9cf7df6-7b49-4194-bf11-16aaca528749, F.Cu at (104.2, 49.4)
- added hex_outline: , clipboard:b9cf7df6-7b49-4194-bf11-16aaca528749, F.Cu at (178.7, 27.9)
- added hex_outline: , clipboard:b9cf7df6-7b49-4194-bf11-16aaca528749, F.Cu at (-32.2, 18.1)
- added hex_outline: , clipboard:b9cf7df6-7b49-4194-bf11-16aaca528749, F.Cu at (141.5, 113.9)
- added hex_outline: , clipboard:b9cf7df6-7b49-4194-bf11-16aaca528749, F.Cu at (-88.0, 28.8)
- added hex_outline: , clipboard:b9cf7df6-7b49-4194-bf11-16aaca528749, F.Cu at (-125.3, 50.3)
- added hex_outline: , clipboard:b9cf7df6-7b49-4194-bf11-16aaca528749, F.Cu at (104.2, 70.9)
- added hex_outline: , clipboard:b9cf7df6-7b49-4194-bf11-16aaca528749, F.Cu at (-106.7, 39.5)
- D10, D11, D12, D13, D14, D15, D16, D17, D18, D19, D20, D21, D22, D4, D5, D6, D7, D8, D9, F1, R6, R7, S1, S10, S11, S12, S13, S14, S15, S16, S17, S18, S19, S2, S20, S3, S4, S5, S6, S7, S8, S9, USBC1: moved to B.Cu
- LED1, LED10, LED11, LED12, LED13, LED14, LED15, LED16, LED17, LED18, LED19, LED2, LED20, LED3, LED4, LED5, LED6, LED7, LED8, LED9: moved to F.Cu
- moved D4 186.1 mm to (220.9, 41.1), turned to 120 degrees
- moved D5 186.1 mm to (220.9, 62.6), turned to 120 degrees
- moved D6 186.1 mm to (220.9, 84.2), turned to 120 degrees
- moved S1 176.1 mm to (215.9, 49.4), turned to -150 degrees
- moved S2 176.1 mm to (215.9, 70.9), turned to -150 degrees
- moved S3 176.1 mm to (215.9, 92.4), turned to -150 degrees
- moved LED2 171.5 mm to (213.6, 66.8), turned to 30 degrees
- moved LED3 171.5 mm to (213.6, 88.3), turned to 30 degrees
- moved LED1 171.5 mm to (213.6, 45.4), turned to 30 degrees
- moved D10 148.7 mm to (202.2, 73.4), turned to 120 degrees
- moved D9 148.7 mm to (202.2, 51.9), turned to 120 degrees
- moved D8 148.7 mm to (202.2, 30.4), turned to 120 degrees
- moved S5 139.0 mm to (197.3, 38.6), turned to -150 degrees
- moved S6 139.0 mm to (197.3, 60.1), turned to -150 degrees
- moved S7 139.0 mm to (197.3, 81.7), turned to -150 degrees
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Connections:
- D11 pad 2: /ROW4 -> /ROW3
- D15 pad 2: /ROW4 -> /ROW2
- D19 pad 2: /ROW4 -> /ROW3
- D2 pad 1: /PWR_BTN -> Net-(D2-Pad1)
- D2 pad 2: Net-(D2-Pad2) -> /PWR_BTN
- D7 pad 2: /ROW4 -> /ROW1
- LED1 pad 1: /LED0 -> /LED1
- LED10 pad 1: /LED9 -> /LED10
- LED11 pad 1: /LED10 -> /LED11
- LED12 pad 1: /LED11 -> /LED12
- LED13 pad 1: /LED12 -> /LED13
- LED14 pad 1: /LED13 -> /LED14
- LED15 pad 1: /LED14 -> /LED15
- LED16 pad 1: /LED15 -> /LED16
- LED17 pad 1: /LED16 -> /LED17
- LED18 pad 1: /LED17 -> /LED18
- LED19 pad 1: /LED18 -> /LED19
- LED2 pad 1: /LED1 -> /LED2
- LED20 pad 1: /LED19 -> /LED20
- LED3 pad 1: /LED2 -> /LED3
- LED4 pad 1: /LED3 -> /LED4
- LED5 pad 1: /LED4 -> /LED5
- LED6 pad 1: /LED5 -> /LED6
- LED7 pad 1: /LED6 -> /LED7
- LED8 pad 1: /LED7 -> /LED8
- LED9 pad 1: /LED8 -> /LED9
- R4 pad 1: Net-(D2-Pad2) -> Net-(D2-Pad1)
- S10 pad 1: Net-(S10-Pad1) -> /COL3
- S11 pad 1: Net-(S10-Pad1) -> /COL3
- S12 pad 1: Net-(S10-Pad1) -> /COL6
- S16 pad 1: /COL4 -> /COL7
- S4 pad 1: /COL1 -> /COL6
- S8 pad 1: /COL2 -> /COL6
- S9 pad 1: Net-(S10-Pad1) -> /COL3
- U2 pad 1: unconnected-(U2-P1.11-Pad1) -> /COL7
- U2 pad 12: unconnected-(U2-P0.26-Pad12) -> /ROW3
- U2 pad 16: /ROW3 -> unconnected-(U2-P0.08-Pad16)
- U2 pad 17: /ROW4 -> /COL6
- U2 pad 28: unconnected-(U2-P15-Pad28) -> /ROW1
- U2 pad 3: /ROW1 -> unconnected-(U2-P0.03-Pad3)
- U2 pad 30: unconnected-(U2-P17-Pad30) -> /COL5
- U2 pad 32: /COL5 -> /COL4
- U2 pad 33: /COL4 -> unconnected-(U2-P0.13-Pad33)
- U2 pad 35: /COL2 -> unconnected-(U2-P0.24-Pad35)
- U2 pad 36: /COL1 -> /COL2
- U2 pad 38: unconnected-(U2-P1.02-Pad38) -> /COL1
- U2 pad 4: unconnected-(U2-AI4-Pad4) -> /ADC
- U2 pad 41: /LED_EN -> /CHRG
- U2 pad 42: /LED_SDA -> unconnected-(U2-P1.06-Pad42)
- U2 pad 43: /LED_SCL -> /STDBY
- U2 pad 7: /ADC -> /LED_EN
- U2 pad 8: /CHRG -> /LED_SDA
- U2 pad 9: /STDBY -> /LED_SCL
- U6 pad 1: /LED19 -> /LED20
- U6 pad 10: /LED8 -> /LED7
- U6 pad 11: /LED9 -> /LED6
- U6 pad 14: /LED12 -> /LED15
- U6 pad 15: /LED13 -> /LED14
- U6 pad 16: /LED14 -> /LED18
- U6 pad 17: /LED15 -> /LED19
- U6 pad 18: /LED16 -> /LED8
- U6 pad 19: /LED17 -> /LED12
- U6 pad 2: /LED0 -> /LED4
- U6 pad 20: /LED18 -> /LED16
- U6 pad 3: /LED1 -> /LED17
- U6 pad 4: /LED2 -> /LED13
- U6 pad 5: /LED3 -> /LED9
- U6 pad 6: /LED4 -> /LED5
- U6 pad 7: /LED5 -> /LED1
- U6 pad 8: /LED6 -> /LED2
- U6 pad 9: /LED7 -> /LED3
- U7 pad 13: GND -> /BAT+
Other:
- copper layers 2 -> 4
