File: kicad/kicad.kicad_sch (KiCad schematic)
At the start: 54 parts, among them Q1 PMF170XP,115, Q2 FS8205A_C2830320, SW1 TS-1088-AR02016, U1 DW01A, U2 BL8573CS8TR, U3 74AHC1G14GW,125, U4 74HC74NS14ARDQ, U5 APTD1608LSECK/J4-PF, U6 CRCW0402787RFKED, U7 NRF52840-QIAA-R7, X1 XTM20032000DT00351005, X2 FC-13532.768KHZ9PF20PPM

Commit message: a lot... almost done schematic... need to rewire to new mcu module... pcb key/led/diode placement done... other componenets tbd
Parts:
- removed C2: 100nF, PCM_JLCPCB:C_0402, symbol PCM_JLCPCB-Capacitors:0402,100nF
- removed L1, L3: CBC3225T100KR, easyeda2kicad:L1210, symbol easyeda2kicad:CBC3225T100KR
- removed R4: RC0402FR-0710KL, easyeda2kicad:R0402, symbol easyeda2kicad:RC0402FR-0710KL
- removed R6: RC0402FR-075K1L, easyeda2kicad:R0402, symbol easyeda2kicad:RC0402FR-075K1L
- removed U3: 74AHC1G14GW,125, easyeda2kicad:SOT-353_L2.1-W1.3-P0.65-LS2.3-BR, symbol easyeda2kicad:74AHC1G14GW,125
- removed U4: 74HC74NS14ARDQ, easyeda2kicad:SOIC-14_L8.7-W3.9-P1.27-LS6.0-BL, symbol easyeda2kicad:74HC74NS14ARDQ
- removed U5: APTD1608LSECK/J4-PF, easyeda2kicad:LED-SMD_L1.6-W0.8-RD, symbol easyeda2kicad:APTD1608LSECK_J4-PF
- removed U6: CRCW0402787RFKED, easyeda2kicad:R0402, symbol easyeda2kicad:FRC0402F1201TS
- added C11: GRM033C71C104KE14D, easyeda2kicad:C0201, symbol easyeda2kicad:GRM033C71C104KE14D
- added C25, C26: GRM155C71C105KE11D, easyeda2kicad:C0402, symbol easyeda2kicad:GRM155C71C105KE11D
- added D10, D11, D12, D13, D14, D15, D16, D17, D18, D19, D20, D21, D22, D4, D5, D6, D7, D8, D9: CDSQC4148-HF, :X1-DFN1006-2_L1.0-W0.6-RD, symbol easyeda2kicad:CDSQC4148-HF
- added L1, L4: BRC2016T100K, :IND-SMD_L2.0-W1.6_BRC2016, symbol easyeda2kicad:BRC2016T100K
- added LED1, LED10, LED11, LED12, LED13, LED14, LED15, LED16, LED17, LED18, LED19, LED2, LED20, LED3, LED4, LED5, LED6, LED7, LED8, LED9: OSO5PAS1C1A-1MA, :LED-SMD_L3.2-W2.8-LS3.5-RD-BLUE, symbol easyeda2kicad:LPT67F-P1R2-35-Z
- added R11: RT0402BRD0737K4L, :R0402, symbol easyeda2kicad:RT0402BRD0737K4L
- added R12, R13, R7: RC0402FR-075K1L, easyeda2kicad:R0402, symbol easyeda2kicad:RC0402FR-075K1L
- added R14: RC0402FR-071ML, easyeda2kicad:R0402, symbol easyeda2kicad:RC0402FR-071ML
- added R9: RC0402FR-0710KL, easyeda2kicad:R0402, symbol easyeda2kicad:RC0402FR-0710KL
- added S1, S10, S11, S12, S13, S14, S15, S16, S17, S18, S19, S2, S20, S3, S4, S5, S6, S7, S8, S9: Choc HEX, hexcaps:PG1350_hotswap, symbol keys:choc_v1_hex
- added U1: 74AHC1G14GW,125, easyeda2kicad:SOT-353_L2.1-W1.3-P0.65-LS2.3-BR, symbol easyeda2kicad:74AHC1G14GW,125
- added U2: E73-2G4M08S1C, :WIRELM-SMD_E73-2G4M08S1C, symbol easyeda2kicad:E73-2G4M08S1C
- added U5: S2B-PH-K-S(LF)(SN), :CONN-TH_S2B-PH-K-S-LF-SN, symbol easyeda2kicad:S2B-PH-K-S(LF)(SN)
- added U6: LP5024RSMR, :VQFN-32_L4.0-W4.0-P0.40-TL-EP, symbol easyeda2kicad:LP5024RSMR
- added U7: SN74HCS74BQAR, :DQFN-14_L3.0-W2.5-P0.50-BL-EP, symbol easyeda2kicad:SN74HCS74BQAR
- NRF1: renamed from U7; footprint easyeda2kicad:AQFN-73_L7.0-W7.0-P0.50-BL-EP4.8 -> Package_DFN_QFN:Nordic_AQFN-73-1EP_7x7mm_P0.5mm
- renumbered C19 to C1, C3 to C10, C23 to C12, C4 to C13, C7 to C14, C6 to C15, C18 to C16, C5 to C17, C9 to C18, C14 to C19, C20 to C2, C17 to C20, C12 to C21, C15 to C22, C16 to C23, C22 to C24, C1 to C3, C11 to C4, C13 to C5, C21 to C6, C10 to C7, C24 to C9, L2 to L3, R7 to R1, R5 to R10, R9 to R2, R10 to R3, R1 to R4, R8 to R5, R2 to R6, R3 to R8, U2 to U3, U1 to U4, X2 to X1, X1 to X2
Connections:
- net P031 is gone; now on net CHRG: NRF1.A8 (P0.31/AIN7)
- net VDD_HV is gone; now on net PWR: C2.1, NRF1.Y2 (VDDH)
- net BAT+: now also S20.1, U1.5 (VCC), U5.1, U7.1 (~{1CLR}), U7.10 (~{2PRE}), U7.14 (VCC), U7.4 (~{1PRE}); no longer D1.A, D2.A, R5.1
- net GND: now also C19.2, NRF1.EP (GND), C11.2, C25.2, C26.2, R11.2, R14.2, R7.2, U1.3 (GND), U5.2, U6.25 (ADDR0), U6.26 (ADDR1), U6.33 (GND), U7.11 (2CLK), U7.12 (2D), U7.13 (~{2CLR}), U7.15 (EP), U7.7 (GND); no longer C19.1, NRF1.0 (GND)
- net P028: no longer R2.1, R3.2
- net PMOS_gate: now also U7.2 (1D), U7.6 (~{1Q})
- net PWR: now also C26.1, LED1.2, LED10.2, LED11.2, LED12.2, LED13.2, LED14.2, LED15.2, LED16.2, LED17.2, LED18.2, LED19.2, LED2.2, LED20.2, LED3.2, LED4.2, LED5.2, LED6.2, LED7.2, LED8.2, LED9.2, U6.27 (VCC); no longer C1.1, C12.1, C15.1, C16.1, C8.1, NRF1.A22 (VDD), NRF1.AD14 (VDD), NRF1.AD23 (VDD), NRF1.B1 (VDD), NRF1.W1 (VDD), R10.2
- net RESET: now also C11.1
- net at USBC1.B5 (CC2): now also R7.1
- net at C10.1, C13.1, C21.2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: now also L4.2
- net at R4.1: now also D2.2; no longer D1.K
- net at NRF1.B3 (DCC): now also L4.1
- net at NRF1.AB2 (DCCH): now also L1.2
- net at C3.1, R4.2: now also D3.2, U1.2 (A); no longer D3.A
- net at L3.1, NRF1.H23 (ANT): now also C19.1; no longer C19.2
- net P004: no longer names the net of NRF1.J1 (P0.04/AIN2)
- net P005: no longer names the net of NRF1.K2 (P0.05/AIN3)
- net P006 renamed ROW3
- net ROW3: now also D10.2, D14.2, D18.2, D22.2, D6.2
- net P007: no longer names the net of NRF1.M2 (P0.07)
- net P008: no longer names the net of NRF1.N1 (P0.08)
- net P011: no longer names the net of NRF1.T2 (P0.11)
- net P012: no longer names the net of NRF1.U1 (P0.12)
- net P029 renamed STDBY
- net STDBY: now also NRF1.B9 (P0.30/AIN6); no longer NRF1.A10 (P0.29/AIN5)
- net P030 renamed CHRG
- net CHRG: now also R9.1; no longer NRF1.B9 (P0.30/AIN6)
- net P101 renamed LED_SDA
- net LED_SDA: now also R12.1, U6.28 (SDA)
- net P102 renamed LED_SCL
- net LED_SCL: now also R13.1, U6.29 (SCL)
- net P103 renamed LED_EN
- net LED_EN: now also R14.1, U6.30 (EN)
- net P108: no longer names the net of NRF1.P2 (P1.08)
- net P109: no longer names the net of NRF1.R1 (P1.09)
- new net: D7.1, S4.2
- new net: D4.1, S1.2
- new net: D1.1, D3.1, R1.1
- new net: D8.1, S5.2
- new net: D10.1, S7.2
- new net: D6.1, S3.2
- new net: D13.1, S10.2
- new net: D11.1, S8.2
- new net: D14.1, S11.2
- new net: S10.1, S11.1, S12.1, S9.1
- new net: D20.1, S17.2
- new net: D9.1, S6.2
- new net: D19.1, S16.2
- new net: D16.1, S13.2
- new net: D18.1, S15.2
- new net: D22.1, S19.2
- new net: D12.1, S9.2
- new net: R11.1, U6.31 (IREF)
- new net: C25.1, U6.32 (VCAP)
- new net: D5.1, S2.2
- new net: D21.1, S18.2
- new net: D15.1, S12.2
- new net: U1.4 (Y), U7.3 (1CLK)
- new net: D17.1, S14.2
- new net ADC: NRF1.A10 (P0.29/AIN5), R2.1, R3.2
- new net COL1: S1.1, S2.1, S3.1, S4.1
- new net COL2: S5.1, S6.1, S7.1, S8.1
- new net COL4: S13.1, S14.1, S15.1, S16.1
- new net COL5: S17.1, S18.1, S19.1
- new net LED0: LED1.1, U6.1 (OUT0)
- new net LED1: LED2.1, U6.2 (OUT1)
- new net LED10: LED11.1, U6.11 (OUT10)
- new net LED11: LED12.1, U6.12 (OUT11)
- new net LED12: LED13.1, U6.13 (OUT12)
- new net LED13: LED14.1, U6.14 (OUT13)
- new net LED14: LED15.1, U6.15 (OUT14)
- new net LED15: LED16.1, U6.16 (OUT15)
- new net LED16: LED17.1, U6.17 (OUT16)
- new net LED17: LED18.1, U6.18 (OUT17)
- new net LED18: LED19.1, U6.19 (OUT18)
- new net LED19: LED20.1, U6.20 (OUT19)
- new net LED2: LED3.1, U6.3 (OUT2)
- new net LED3: LED4.1, U6.4 (OUT3)
- new net LED4: LED5.1, U6.5 (OUT4)
- new net LED5: LED6.1, U6.6 (OUT5)
- new net LED6: LED7.1, U6.7 (OUT6)
- new net LED7: LED8.1, U6.8 (OUT7)
- new net LED8: LED9.1, U6.9 (OUT8)
- new net LED9: LED10.1, U6.10 (OUT9)
- new net PWR_BTN: D1.2, D2.1, S20.2
- new net ROW1: D12.2, D16.2, D20.2, D4.2, D8.2
- new net ROW2: D13.2, D17.2, D21.2, D5.2, D9.2
- new net ROW4: D11.2, D15.2, D19.2, D7.2
- new net VDD_nRF: C1.1, C12.1, C15.1, C16.1, C8.1, L1.1, NRF1.A22 (VDD), NRF1.AD14 (VDD), NRF1.AD23 (VDD), NRF1.B1 (VDD), NRF1.W1 (VDD), R10.2, R12.2, R13.2, R5.1, R9.2
Other:
- note removed: "ON + battery low LED indicator"
- moved on the sheet: C19, C20, C3, Q2, R1, R2, R3, R4, R5, SW1, U4

Commit message: changed raw mcu to e73module with antena... cleaned pcb a little
Parts:
- removed C1, C2, C6, C9: GRM188C71C475KE21D, easyeda2kicad:C0603, symbol easyeda2kicad:GRM188C71C475KE21D
- removed C10, C8: GRM155C71C105KE11D, easyeda2kicad:C0402, symbol easyeda2kicad:GRM155C71C105KE11D
- removed C12, C15, C16, C7: GRM033C71C104KE14D, easyeda2kicad:C0201, symbol easyeda2kicad:GRM033C71C104KE14D
- removed C13: CL05B473KO5NNNC, easyeda2kicad:C0402, symbol easyeda2kicad:CL05B473KO5NNNC
- removed C14, C21: N.C., easyeda2kicad:C0402, symbol easyeda2kicad:0402CG120F500NT
- removed C17, C18, C4, C5: 0402CG120F500NT, easyeda2kicad:C0402, symbol easyeda2kicad:0402CG120F500NT
- removed C19: GJM1555C1HR80WB01D, easyeda2kicad:C0402, symbol easyeda2kicad:GJM1555C1HR80WB01D
- removed C20: GRM1555C1H821FA01D, easyeda2kicad:C0402, symbol easyeda2kicad:GRM1555C1H821FA01D
- removed C22: GJM1555C1HR50WB01D, easyeda2kicad:C0402, symbol easyeda2kicad:GJM1555C1HR50WB01D
- removed C23: N.C, easyeda2kicad:C0402, symbol easyeda2kicad:GJM1555C1HR50WB01D
- removed C24: GCM1555C1H101FA16D, easyeda2kicad:C0402, symbol easyeda2kicad:GCM1555C1H101FA16D
- removed L3: 0402DC-4N7XJRW, easyeda2kicad:IND-SMD_L1.1-W0.6, symbol easyeda2kicad:0402DC-4N7XJRW
- removed L4: BRC2016T100K, :IND-SMD_L2.0-W1.6_BRC2016, symbol easyeda2kicad:BRC2016T100K
- removed NRF1: NRF52840-QIAA-R7, Package_DFN_QFN:Nordic_AQFN-73-1EP_7x7mm_P0.5mm, symbol easyeda2kicad:NRF52840-QIAA-R7
- removed X1: FC-13532.768KHZ9PF20PPM, easyeda2kicad:OSC-SMD_L3.2-W1.5, symbol easyeda2kicad:FC-13532.768KHZ9PF20PPM
- removed X2: XTM20032000DT00351005, easyeda2kicad:CRYSTAL-SMD_4P-L2.0-W1.6-BL-A, symbol easyeda2kicad:XTM20032000DT00351005
- added C27: GRM188C71C475KE21D, easyeda2kicad:C0603, symbol easyeda2kicad:GRM188C71C475KE21D
- added C28, C29: 0402CG120F500NT, easyeda2kicad:C0402, symbol easyeda2kicad:0402CG120F500NT
- added X3: FC-13532.768KHZ9PF20PPM, easyeda2kicad:OSC-SMD_L3.2-W1.5, symbol easyeda2kicad:FC-13532.768KHZ9PF20PPM
Connections:
- net ADC: now also U2.7 (AI0)
- net CHRG: now also U2.8 (AI5)
- net COL1: now also U2.36 (P1.00)
- net COL2: now also U2.35 (P0.24)
- net COL3: now also U2.34 (P0.22)
- net COL4: now also U2.33 (P0.13)
- net COL5: now also U2.32 (P0.20)
- net D+: now also U2.31 (D+)
- net D-: now also U2.29 (D-)
- net GND: now also U2.21 (GND), U2.24 (GND), U2.5 (GND), C27.2, C28.2, C29.2
- net LED0: now also U6.2 (OUT1); no longer U6.1 (OUT0)
- net LED1: now also U6.3 (OUT2); no longer U6.2 (OUT1)
- net LED10: now also U6.12 (OUT11); no longer U6.11 (OUT10)
- net LED11: now also U6.13 (OUT12); no longer U6.12 (OUT11)
- net LED12: now also U6.14 (OUT13); no longer U6.13 (OUT12)
- net LED13: now also U6.15 (OUT14); no longer U6.14 (OUT13)
- net LED14: now also U6.16 (OUT15); no longer U6.15 (OUT14)
- net LED15: now also U6.17 (OUT16); no longer U6.16 (OUT15)
- net LED16: now also U6.18 (OUT17); no longer U6.17 (OUT16)
- net LED17: now also U6.19 (OUT18); no longer U6.18 (OUT17)
- net LED18: now also U6.20 (OUT19); no longer U6.19 (OUT18)
- net LED19: now also U6.1 (OUT0); no longer U6.20 (OUT19)
- net LED2: now also U6.4 (OUT3); no longer U6.3 (OUT2)
- net LED3: now also U6.5 (OUT4); no longer U6.4 (OUT3)
- net LED4: now also U6.6 (OUT5); no longer U6.5 (OUT4)
- net LED5: now also U6.7 (OUT6); no longer U6.6 (OUT5)
- net LED6: now also U6.8 (OUT7); no longer U6.7 (OUT6)
- net LED7: now also U6.9 (OUT8); no longer U6.8 (OUT7)
- net LED8: now also U6.10 (OUT9); no longer U6.9 (OUT8)
- net LED9: now also U6.11 (OUT10); no longer U6.10 (OUT9)
- net LED_EN: now also U2.41 (NF1)
- net LED_SCL: now also U2.43 (NF2)
- net LED_SDA: now also U2.42 (P1.06)
- net PWR: now also U2.23 (VDH)
- net RESET: now also U2.26 (RST)
- net ROW1: now also U2.3 (P0.03)
- net ROW2: now also U2.14 (P0.06)
- net ROW3: now also U2.16 (P0.08)
- net ROW4: now also U2.17 (P1.09)
- net STDBY: now also U2.9 (AI7)
- net SWBCLK: now also U2.39 (SWC)
- net SWDIO: now also U2.37 (SWD)
- net VBUS: now also F1.2, U2.27 (VBS), U3.4 (VCC), C27.1; no longer F1.1, USBC1.A4B9 (VBUS), USBC1.B4A9 (VBUS)
- net VDD_nRF: now also L1.2, U2.19 (VCC); no longer L1.1
- net at U2.11 (XL1): now also C28.1, X3.1
- net at U2.13 (XL2): now also C29.1, X3.2
- net at U2.25 (DCH): now also L1.1
- new net: F1.1, USBC1.A4B9 (VBUS), USBC1.B4A9 (VBUS)
Other:
- moved on the sheet: C11, F1, L1, R2, R3, R5, SW1, U2

Commit message: ...
Connections:
- net ADC: now also U2.4 (AI4); no longer U2.7 (AI0)
- net BAT+: now also U7.13 (~{2CLR})
- net CHRG: now also U2.41 (NF1); no longer U2.8 (AI5)
- net COL1: now also U2.38 (P1.02); no longer S4.1, U2.36 (P1.00)
- net COL2: now also U2.36 (P1.00); no longer S8.1, U2.35 (P0.24)
- net COL3: now also S10.1, S11.1, S9.1
- net COL4: now also U2.32 (P0.20); no longer S16.1, U2.33 (P0.13)
- net COL5: now also U2.30 (P17); no longer U2.32 (P0.20)
- net GND: no longer U7.13 (~{2CLR})
- net LED1: now also LED1.1, U6.7 (OUT6); no longer LED2.1, U6.3 (OUT2)
- net LED10: now also LED10.1; no longer LED11.1
- net LED11: now also LED11.1; no longer LED12.1
- net LED12: now also LED12.1, U6.19 (OUT18); no longer LED13.1, U6.14 (OUT13)
- net LED13: now also LED13.1, U6.4 (OUT3); no longer LED14.1, U6.15 (OUT14)
- net LED14: now also LED14.1, U6.15 (OUT14); no longer LED15.1, U6.16 (OUT15)
- net LED15: now also LED15.1, U6.14 (OUT13); no longer LED16.1, U6.17 (OUT16)
- net LED16: now also LED16.1, U6.20 (OUT19); no longer LED17.1, U6.18 (OUT17)
- net LED17: now also LED17.1, U6.3 (OUT2); no longer LED18.1, U6.19 (OUT18)
- net LED18: now also LED18.1, U6.16 (OUT15); no longer LED19.1, U6.20 (OUT19)
- net LED19: now also LED19.1, U6.17 (OUT16); no longer LED20.1, U6.1 (OUT0)
- net LED2: now also LED2.1, U6.8 (OUT7); no longer LED3.1, U6.4 (OUT3)
- net LED3: now also LED3.1, U6.9 (OUT8); no longer LED4.1, U6.5 (OUT4)
- net LED4: now also LED4.1, U6.2 (OUT1); no longer LED5.1, U6.6 (OUT5)
- net LED5: now also LED5.1, U6.6 (OUT5); no longer LED6.1, U6.7 (OUT6)
- net LED6: now also LED6.1, U6.11 (OUT10); no longer LED7.1, U6.8 (OUT7)
- net LED7: now also LED7.1, U6.10 (OUT9); no longer LED8.1, U6.9 (OUT8)
- net LED8: now also LED8.1, U6.18 (OUT17); no longer LED9.1, U6.10 (OUT9)
- net LED9: now also LED9.1, U6.5 (OUT4); no longer LED10.1, U6.11 (OUT10)
- net LED_EN: now also U2.7 (AI0); no longer U2.41 (NF1)
- net LED_SCL: now also U2.9 (AI7); no longer U2.43 (NF2)
- net LED_SDA: now also U2.8 (AI5); no longer U2.42 (P1.06)
- net PWR_BTN: now also D2.2; no longer D2.1
- net ROW1: now also D7.2, U2.28 (P15); no longer U2.3 (P0.03)
- net ROW2: now also D15.2
- net ROW3: now also D11.2, D19.2, U2.12 (P0.26); no longer U2.16 (P0.08)
- net STDBY: now also U2.43 (NF2); no longer U2.9 (AI7)
- net at R4.1: now also D2.1; no longer D2.2
- net COL7: now reaches U2.1 (P1.11)
- net COL7: now also S16.1
- removed net LED0: LED1.1, U6.2 (OUT1)
- removed net ROW4: D11.2, D15.2, D19.2, D7.2, U2.17 (P1.09)
- new net COL6: S12.1, S4.1, S8.1, U2.17 (P1.09)
- new net LED20: LED20.1, U6.1 (OUT0)
Other:
- moved on the sheet: C25, C26, D10, D11, D12, D13, D14, D15, D16, D17, D18, D19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

Commit message: psb outline
Connections:
- net LED1: now also U6.18 (OUT17); no longer U6.7 (OUT6)
- net LED10: now also U6.13 (OUT12); no longer U6.12 (OUT11)
- net LED11: now also U6.6 (OUT5); no longer U6.13 (OUT12)
- net LED12: now also U6.2 (OUT1); no longer U6.19 (OUT18)
- net LED13: now also U6.21 (OUT20); no longer U6.4 (OUT3)
- net LED14: now also U6.14 (OUT13); no longer U6.15 (OUT14)
- net LED15: now also U6.5 (OUT4); no longer U6.14 (OUT13)
- net LED16: now also U6.1 (OUT0); no longer U6.20 (OUT19)
- net LED17: now also U6.22 (OUT21); no longer U6.3 (OUT2)
- net LED18: now also U6.17 (OUT16); no longer U6.16 (OUT15)
- net LED19: now also U6.4 (OUT3); no longer U6.17 (OUT16)
- net LED2: now also U6.11 (OUT10); no longer U6.8 (OUT7)
- net LED20: now also U6.24 (OUT23); no longer U6.1 (OUT0)
- net LED3: now also U6.8 (OUT7); no longer U6.9 (OUT8)
- net LED4: now also U6.23 (OUT22); no longer U6.2 (OUT1)
- net LED5: now also U6.19 (OUT18); no longer U6.6 (OUT5)
- net LED6: now also U6.12 (OUT11); no longer U6.11 (OUT10)
- net LED7: now also U6.7 (OUT6); no longer U6.10 (OUT9)
- net LED8: now also U6.3 (OUT2); no longer U6.18 (OUT17)
- net LED9: now also U6.20 (OUT19); no longer U6.5 (OUT4)

Commit message: .
Parts:
- removed D1, D2: NSR05F20NXT5G, easyeda2kicad:DSN2_L1.0-W0.6-RD, symbol easyeda2kicad:NSR05F20NXT5G
- removed U1: 74AHC1G14GW,125, easyeda2kicad:SOT-353_L2.1-W1.3-P0.65-LS2.3-BR, symbol easyeda2kicad:74AHC1G14GW,125
- added R15: RC0402FR-074M3L, :R0402, symbol easyeda2kicad:RC0402FR-074M3L
- added R16: RC0402FR-071ML, easyeda2kicad:R0402, symbol easyeda2kicad:RC0402FR-071ML
- added U1: TLV7031QDCKRQ1, :SC-70-5_L2.0-W1.3-P0.65-LS2.1-BR, symbol easyeda2kicad:TLV7031QDCKRQ1
Connections:
- net GND: now also R15.2, U1.2 (VEE)
- net PWR_BTN: now also D3.1, R1.1, R4.1, R16.1, U1.5 (VCC)
- net at C3.1, D3.2, R4.2: now also U1.3 (IN+)
- net at U7.3 (1CLK): now also U1.1 (OUT)
- new net: R15.1, R16.2, U1.4 (IN-)
Other:
- moved on the sheet: C3, D3, R1, R4

Commit message: ...
Parts:
- added C10, C11, C12, C13, C14, C15, C16, C17, C18, C19, C20, C21, C22, C23, C24, C25, C26, C27, C8, C9: GRM033C71C104KE14D, easyeda2kicad:C0201, symbol easyeda2kicad:GRM033C71C104KE14D
- renumbered C3 to C1, C11 to C2, C27 to C3, C28 to C4, C29 to C5, C25 to C6, C26 to C7, D3 to D1, D13 to D10, D17 to D11, D21 to D12, D15 to D13, D6 to D14, D10 to D15, D14 to D16, D18 to D17, D22 to D18, D11 to D19, D4 to D2, D19 to D20, D8 to D3, D12 to D4, D16 to D5, D20 to D6, D5 to D8, LED17 to LED10, LED4 to LED11, LED14 to LED12, LED11 to LED13, LED8 to LED14, LED18 to LED15, LED15 to LED16, LED12 to LED17, LED19 to LED18, LED16 to LED19, LED5 to LED2, LED2 to LED3, LED9 to LED4, LED6 to LED5, LED3 to LED6, LED13 to LED7, LED10 to LED8, LED7 to LED9, R4 to R1, R5 to R10, R2 to R11, R3 to R12, R11 to R13, R12 to R14, R13 to R15, R14 to R16, R6 to R2, R8 to R3, R9 to R4, R10 to R5, R1 to R6, R15 to R8, R16 to R9, S14 to S11, S18 to S12, S12 to S13, S3 to S14, S7 to S15, S11 to S16, S15 to S17, S19 to S18, S8 to S19, S5 to S2, S16 to S20, S9 to S3, S13 to S4, S17 to S5, S4 to S6, S20 to S7, S2 to S8, S6 to S9, U4 to U1, U3 to U2, U1 to U3, U7 to U4, U2 to U6, U6 to U7, X3 to X1
Connections:
- net GND: now also C10.2, C11.2, C12.2, C13.2, C14.2, C15.2, C16.2, C17.2, C18.2, C19.2, C20.2, C21.2, C22.2, C23.2, C24.2, C25.2, C26.2, C27.2, C8.2, C9.2
- net PWR: now also C10.1, C11.1, C12.1, C13.1, C14.1, C15.1, C16.1, C17.1, C18.1, C19.1, C20.1, C21.1, C22.1, C23.1, C24.1, C25.1, C26.1, C27.1, C8.1, C9.1
Other:
- moved on the sheet: C6, C7, D10, D11, D12, D13, D14, D15, D16, D17, D18, D19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

Commit message: ... started doing wiring
Parts:
- renumbered C20 to C11, C11 to C12, C21 to C13, C12 to C14, C22 to C15, C13 to C16, C23 to C17, C14 to C18, C24 to C19, C4 to C2, C15 to C20, C25 to C21, C16 to C22, C26 to C23, C17 to C24, C27 to C25, C6 to C26, C7 to C27, C5 to C3, C2 to C4, C3 to C5, C8 to C6, C18 to C7, C9 to C8, C19 to C9, D16 to D10, D5 to D11, D11 to D12, D17 to D13, D6 to D14, D12 to D15, D18 to D16, D7 to D17, D13 to D18, D8 to D3, D14 to D4, D3 to D5, D9 to D6, D15 to D7, D4 to D8, D10 to D9, LED8 to LED10, LED13 to LED11, LED17 to LED12, LED7 to LED13, LED12 to LED14, LED16 to LED15, LED19 to LED16, LED10 to LED17, LED15 to LED18, LED18 to LED19, LED3 to LED2, LED6 to LED3, LED11 to LED4, LED2 to LED5, LED5 to LED6, LED9 to LED7, LED14 to LED8, LED4 to LED9, R6 to R1, R3 to R10, R4 to R11, R5 to R12, R1 to R2, R8 to R3, R11 to R4, R12 to R5, R9 to R6, R10 to R7, R2 to R8, R7 to R9, S4 to S10, S17 to S12, S5 to S13, S12 to S14, S18 to S15, S6 to S16, S13 to S17, S19 to S18, S20 to S19, S8 to S2, S7 to S20, S14 to S3, S2 to S4, S9 to S5, S15 to S6, S3 to S7, S10 to S8, S16 to S9, U3 to U1, U6 to U2, U4 to U3, U2 to U4, U1 to U5, U5 to U6
Other:
- moved on the sheet: C10, C11, C12, C13, C14, C15, C16, C17, C18, C19, C20, C21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

Commit message: finished part placement and wiring. TODO: wire swd pins. mirror the board for left side.
Parts:
- removed U3: SN74HCS74BQAR, :DQFN-14_L3.0-W2.5-P0.50-BL-EP, symbol easyeda2kicad:SN74HCS74BQAR
- added U3: SN74LVC1G74DQER, :X2SON-8_L1.4-W1.0-P0.35-BL, symbol easyeda2kicad:SN74LVC1G74DQER
Connections:
- net BAT+: now also U3.6 (~{CLR}), U3.7 (~{PRE}), U3.8 (VCC)
- net CHRG: now also U2.43 (NF2); no longer U2.41 (NF1)
- net GND: now also U3.4 (GND)
- net PMOS_gate: now also U3.2 (D), U3.3 (~{Q})
- net STDBY: now also U2.41 (NF1); no longer U2.43 (NF2)
- net at U1.1 (OUT): now also U3.1 (CLK)
Other:
- moved on the sheet: C10, C11, C12, C13, C14, C15, C16, C17, C18, C19, C2, C20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
