File: kicad/kicad.kicad_sch (KiCad schematic)
At the start: 117 parts, among them Q1 PMF170XP,115, Q2 FS8205A_C2830320, SW1 TS-1088-AR02016, U1 TLV7031QDCKRQ1, U2 E73-2G4M08S1C, U3 SN74LVC1G74DQER, U4 BL8573CS8TR, U5 DW01A, U6 S2B-PH-K-S(LF)(SN), U7 LP5024RSMR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

Commit message: .
Parts:
- added H1: HC-PM254-8.5H-1X3PW, :HDR-TH_3P-P2.54_HC-PM254-8.5H-1X3PW, symbol easyeda2kicad:HC-PM254-8.5H-1X3PW
Connections:
- net GND: now also H1.1
- net SWBCLK: now also H1.2
- net SWDIO: now also H1.3
Other:
- note added: "Charging and battery"
- note added: "Debug Connector"
- note added: "Key Matrix"
- note added: "LED Matrix"
- note added: "MCU"
- note added: "ON/OFF Circuit"
- note added: "Reset Button"
- note removed: "ON/OFF"
- moved on the sheet: C10, C11, C12, C13, C14, C15, C16, C17, C18, C19, C2, C20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

Commit message: added art... and some other stuff
Parts:
- removed U5: DW01A, Package_TO_SOT_SMD:SOT-23-6, symbol Battery_Management:DW01A
- added U8: DW01A_C42380662, :SOT-23-6_L2.9-W1.6-P0.95-LS2.9-BL, symbol easyeda2kicad:DW01A_C42380662
Connections:
- net BAT+: now also U8.6 (VSS)
- net GND: now also U8.5 (VDD)
- net LED10: now also U7.21 (OUT20); no longer U7.13 (OUT12)
- net LED11: now also U7.14 (OUT13); no longer U7.6 (OUT5)
- net LED12: now also U7.5 (OUT4); no longer U7.2 (OUT1)
- net LED13: now also U7.22 (OUT21); no longer U7.21 (OUT20)
- net LED14: now also U7.17 (OUT16); no longer U7.14 (OUT13)
- net LED15: now also U7.4 (OUT3); no longer U7.5 (OUT4)
- net LED16: now also U7.23 (OUT22); no longer U7.1 (OUT0)
- net LED17: now also U7.2 (OUT1); no longer U7.22 (OUT21)
- net LED18: now also U7.3 (OUT2); no longer U7.17 (OUT16)
- net LED19: now also U7.1 (OUT0); no longer U7.4 (OUT3)
- net LED4: now also U7.19 (OUT18); no longer U7.23 (OUT22)
- net LED5: now also U7.12 (OUT11); no longer U7.19 (OUT18)
- net LED6: now also U7.7 (OUT6); no longer U7.12 (OUT11)
- net LED7: now also U7.20 (OUT19); no longer U7.7 (OUT6)
- net LED8: now also U7.13 (OUT12); no longer U7.3 (OUT2)
- net LED9: now also U7.6 (OUT5); no longer U7.20 (OUT19)
- net at Q2.2 (D1/D2), Q2.5 (D1/D2): now also U8.2 (VM)
- net at Q2.4 (G2): now also U8.1 (DO)
- net at Q2.6 (G1): now also U8.3 (CO)
Other:
- moved on the sheet: R14, R15, R16
