File: kicad/panel.kicad_pcb (KiCad board)
At the start: 4 copper layers, 273 x 119.9 mm, 234 parts, among them Q1 PMF170XP,115, Q2 FS8205A_C2830320, SW1 TS-1088-AR02016, U1 SN74LVC1G17DBVR, U10 SN74LVC1G74DQER, U2 E73-2G4M08S1C, U3 SN74LVC1G74DQER, U4 S2B-PH-K-S(LF)(SN), U5 BL8573CS8TR, U6 DW01A_C42380662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

Commit message: ... todo: update panel woth newest left and right pcb
Parts:
- removed the C6 at (59.0, 79.5)
- removed the C6 at (295.4, 93.2)
- removed the R8 at (65.7, 82.2)
- removed the R8 at (292.9, 93.2)
- removed the REF** at (252.5, 99.6)
- removed the REF** at (233.9, 45.9)
- removed the REF** at (196.7, 67.4)
- removed the SW1 at (62.9, 79.8)
- removed the SW1 at (294.0, 91.0)
- added C6: CL05B104KB54PNC, easyeda2kicad:C0402, F.Cu at (295.4, 93.2)
- added C6: CL05B104KB54PNC, easyeda2kicad:C0402, F.Cu at (59.3, 79.6)
- added R8: 0402WGF1002TCE, easyeda2kicad:R0402, F.Cu at (65.4, 82.3)
- added R8: 0402WGF1002TCE, easyeda2kicad:R0402, F.Cu at (292.9, 93.2)
- added REF**: MountingHole_2.2mm_M2, MountingHole:MountingHole_2.2mm_M2, F.Cu at (233.9, 45.9)
- added REF**: MountingHole_2.2mm_M2, MountingHole:MountingHole_2.2mm_M2, F.Cu at (252.5, 99.6)
- added REF**: MountingHole_2.2mm_M2, MountingHole:MountingHole_2.2mm_M2, F.Cu at (196.7, 67.4)
- added SW1: TS-1088-AR02016, easyeda2kicad:SW-SMD_L3.9-W3.0-P4.45, F.Cu at (63.4, 79.4)
- added SW1: TS-1088-AR02016, easyeda2kicad:SW-SMD_L3.9-W3.0-P4.45, F.Cu at (294.0, 91.0)
- R1: value RC0402FR-071ML -> 0402WGF1004TCE
- R3, R5: value RC0402FR-07100KL -> 0402WGF1002TCE
Routing:
- net /VDD_nRF: track 151.2 -> 152.2 mm
- net /RESET: track 27.0 -> 27.6 mm
- net GND: vias 479 -> 481
