File: kicad/right.kicad_sch (KiCad schematic)
At the start: 101 parts, among them Q1 PMF170XP,115, Q2 FS8205A_C2830320, SW1 TS-1088-AR02016, U1 SN74LVC1G17DBVR, U2 E73-2G4M08S1C, U3 SN74LVC1G74DQER, U4 S2B-PH-K-S(LF)(SN), U5 BL8573CS8TR, U6 DW01A_C42380662, U7 LP5024RSMR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

Commit message: changed on/off timing resistor to 2M61 0805
Parts:
- removed R6: 0402WGF1604TCE, easyeda2kicad:R0402, symbol easyeda2kicad:0402WGF1604TCE
- added R5: RC0805FR-072M61L, easyeda2kicad:R0805, symbol easyeda2kicad:RC0805FR-072M61L
Connections:
- net PWR_BTN: now also R5.1
- net at C2.1, D1.2, U1.2 (A): now also R5.2
Changed lines of the file:
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@@
-	)
-	(symbol
-		(lib_id "easyeda2kicad:0402WGF1604TCE")
-		(at 327.66 120.65 0)
-		(unit 1)
-		(body_style 1)
-		(exclude_from_sim no)
-		(in_bom yes)
-		(on_board yes)
-		(in_pos_files yes)
-		(dnp no)
-		(fields_autoplaced yes)
-		(property "Reference" "R6"
-			(at 327.66 118.11 0)
-			(show_name no)
-			(do_not_autoplace no)
-			(effects
-				(font
-					(size 1.27 1.27)
-				)
-			)
-		)
-		(property "Value" "0402WGF1604TCE"
-			(at 327.66 116.84 0)
-			(hide yes)
-			(show_name no)
-			(do_not_autoplace no)
-			(effects
-				(font
-					(size 1.27 1.27)
-				)
-			)
-		)
-		(property "Footprint" "easyeda2kicad:R0402"
-			(at 327.66 128.27 0)
-			(hide yes)
-			(show_name no)
-			(do_not_autoplace no)
-			(effects
-				(font
-					(size 1.27 1.27)
-				)
-			)
-		)
-		(property "Datasheet" "https://lcsc.com/product-detail/Chip-Resistor-Surface-Mount_Uniroyal-Elec-0402WGF1604TCE_C423231.html"
-			(at 327.66 130.81 0)
-			(hide yes)
-			(show_name no)
-			(do_not_autoplace no)
-			(effects
-				(font
-					(size 1.27 1.27)
-				)
-			)
-		)
-		(property "Description" "3M48"
-			(at 327.66 120.65 0)
-			(show_name no)
-			(do_not_autoplace no)
-			(effects
-				(font
-					(size 1.016 1.016)
-				)
-			)
-		)
-		(property "LCSC Part" "C423231"
-			(at 327.66 133.35 0)
-			(hide yes)
-			(show_name no)
-			(do_not_autoplace no)
-			(effects
-				(font
-					(size 1.27 1.27)
-				)
-			)
-		)
-		(pin "2"
-		)
-		(pin "1"
-		)
-		(instances
-			(project "right"
-				(path "/3171f1b4-f2dd-4471-8b63-415e18370dba"
-					(reference "R6")
-					(unit 1)
-				)
-			)
-		)
 	)
 	(symbol
@@
 					(unit 1)
 				)
+			)
+		)
+	)
+	(symbol
+		(lib_id "easyeda2kicad:RC0805FR-072M61L")
+		(at 327.66 120.65 0)
+		(unit 1)
+		(body_style 1)
+		(exclude_from_sim no)
+		(in_bom yes)
+		(on_board yes)
+		(in_pos_files yes)
+		(dnp no)
+		(fields_autoplaced yes)
+		(property "Reference" "R5"
+			(at 327.66 114.3 0)
+			(show_name no)
+			(do_not_autoplace no)
+			(effects
+				(font
+					(size 1.27 1.27)
+				)
+			)
+		)
+		(property "Value" "RC0805FR-072M61L"
+			(at 327.66 116.84 0)
+			(show_name no)
+			(do_not_autoplace no)
+			(effects
+				(font
+					(size 1.27 1.27)
+				)
+			)
+		)
+		(property "Footprint" "easyeda2kicad:R0805"
+			(at 327.66 128.27 0)
+			(hide yes)
+			(show_name no)
+			(do_not_autoplace no)
+			(effects
+				(font
+					(size 1.27 1.27)
+				)
+			)
+		)
+		(property "Datasheet" "https://lcsc.com/product-detail/New-Arrivals_YAGEO-RC0805FR-072M61L_C483050.html"
+			(at 327.66 130.81 0)
+			(hide yes)
+			(show_name no)
+			(do_not_autoplace no)
+			(effects
+				(font
+					(size 1.27 1.27)
+				)
+			)
+		)
+		(property "Description" "2M61"
+			(at 327.66 120.65 0)
+			(show_name no)
+			(do_not_autoplace no)
+			(effects
+				(font
+					(size 1.143 1.143)
+				)
+			)
+		)
+		(property "Manufacturer" "YAGEO(国巨)"
+			(at 327.66 133.35 0)
+			(hide yes)
+			(show_name no)
+			(do_not_autoplace no)
+			(effects
+				(font
+					(size 1.27 1.27)
+				)
+			)
+		)
+		(property "MPN" "RC0805FR-072M61L"
+			(at 327.66 135.89 0)
+			(hide yes)
+			(show_name no)
+			(do_not_autoplace no)
+			(effects
+				(font
+					(size 1.27 1.27)
+				)
+			)
+		)
+		(property "LCSC Part" "C483050"
+			(at 327.66 138.43 0)
+			(hide yes)
+			(show_name no)
+			(do_not_autoplace no)
+			(effects
+				(font
+					(size 1.27 1.27)
+				)
+			)
+		)
+		(pin "1"
+		)
+		(pin "2"
+		)
+		(instances
+			(project "right"
+				(path "/3171f1b4-f2dd-4471-8b63-415e18370dba"
+					(reference "R5")
+					(unit 1)
+				)

Commit message: added gnd vias all over the board. went trough schematic again. changed resistor for rc to bigger one in footprint, and smaller one in Ohm. both left and right sides are ready. just need to go over the kicads check and lastly let someone on discord have a look on the project
Parts:
- removed R15: RT0402BRD0737K4L, :R0402, symbol easyeda2kicad:RT0402BRD0737K4L
- added R6: ERA2AED753X, easyeda2kicad:R0402, symbol easyeda2kicad:ERA2AED753X
Connections:
- net BAT+: now also U6.5 (VDD); no longer U6.6 (VSS)
- net GND: now also U6.6 (VSS), R6.2; no longer U6.5 (VDD)
- net at U7.31 (IREF): now also R6.1
- no-connect marks 0 -> 20
Changed lines of the file:
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@@
 		(color 0 0 0 0)
 	)
+	(no_connect
+		(at 280.67 33.02)
+	)
+	(no_connect
+		(at 313.69 71.12)
+	)
+	(no_connect
+		(at 160.02 49.53)
+	)
+	(no_connect
+		(at 298.45 71.12)
+	)
+	(no_connect
+		(at 271.78 184.15)
+	)
+	(no_connect
+		(at 160.02 52.07)
+	)
+	(no_connect
+		(at 340.36 29.21)
+	)
+	(no_connect
+		(at 340.36 46.99)
+	)
+	(no_connect
+		(at 280.67 38.1)
+	)
+	(no_connect
+		(at 280.67 40.64)
+	)
+	(no_connect
+		(at 134.62 49.53)
+	)
+	(no_connect
+		(at 280.67 35.56)
+	)
+	(no_connect
+		(at 280.67 48.26)
+	)
+	(no_connect
+		(at 271.78 199.39)
+	)
+	(no_connect
+		(at 260.35 236.22)
+	)
+	(no_connect
+		(at 349.25 187.96)
+	)
+	(no_connect
+		(at 340.36 41.91)
+	)
+	(no_connect
+		(at 372.11 187.96)
+	)
+	(no_connect
+		(at 280.67 50.8)
+	)
+	(no_connect
+		(at 340.36 24.13)
+	)
 	(bus_entry
 		(at 166.37 59.69)
@@
 		)
 	)
-	(wire
-		(pts
-			(xy 260.35 243.84) (xy 260.35 241.3)
-		)
-		(stroke
-			(width 0)
-			(type default)
-		)
-	)
 	(bus
 		(pts
@@
 		)
 	)
-	(label "BAT+"
-		(at 260.35 243.84 180)
-		(effects
-			(font
-				(size 1.27 1.27)
-			)
-			(justify right bottom)
-		)
-	)
 	(label "LED5"
 		(at 134.62 57.15 180)
@@
 		)
 	)
+	(label "BAT+"
+		(at 260.35 238.76 180)
+		(effects
+			(font
+				(size 1.27 1.27)
+			)
+			(justify right bottom)
+		)
+	)
 	(label "BAT_ALTR"
 		(at 372.11 242.57 270)
@@
 	)
 	(symbol
-		(lib_id "PCM_SparkFun-PowerSymbol:GND")
-		(at 260.35 238.76 270)
-		(unit 1)
-		(body_style 1)
-		(exclude_from_sim no)
-		(in_bom yes)
-		(on_board yes)
-		(in_pos_files yes)
-		(dnp no)
-		(fields_autoplaced yes)
-		(property "Reference" "#PWR022"
-			(at 254 238.76 0)
-			(hide yes)
-			(show_name no)
-			(do_not_autoplace no)
-			(effects
-				(font
-					(size 1.27 1.27)
-				)
-			)
-		)
-		(property "Value" "GND"
-			(at 256.54 238.76 0)
-			(show_name no)
-			(do_not_autoplace yes)
-			(effects
-				(font
-					(size 1.27 1.27)
-				)
-			)
-		)
-		(property "Footprint" ""
-			(at 260.35 238.76 0)
-			(hide yes)
-			(show_name no)
-			(do_not_autoplace no)
-			(effects
-				(font
-					(size 1.27 1.27)
-				)
-			)
-		)
-		(property "Datasheet" ""
-			(at 260.35 238.76 0)
-			(hide yes)
-			(show_name no)
-			(do_not_autoplace no)
-			(effects
-				(font
-					(size 1.27 1.27)
-				)
-			)
-		)
-		(property "Description" "Power symbol creates a global label with name \"GND\" , ground"
-			(at 251.46 238.76 0)
-			(hide yes)
-			(show_name no)
-			(do_not_autoplace no)
-			(effects
-				(font
-					(size 1.27 1.27)
-				)
-			)
-		)
-		(pin "1"
-		)
-		(instances
-			(project "right"
-				(path "/3171f1b4-f2dd-4471-8b63-415e18370dba"
-					(reference "#PWR022")
-					(unit 1)
-				)
-			)
-		)
-	)
-	(symbol
 		(lib_id "keys:choc_v1_hex")
 		(at 74.93 199.39 0)
@@
 	)
 	(symbol
+		(lib_id "easyeda2kicad:ERA2AED753X")
+		(at 195.58 31.75 0)
+		(unit 1)
+		(body_style 1)
+		(exclude_from_sim no)
+		(in_bom yes)
+		(on_board yes)
+		(in_pos_files yes)
+		(dnp no)
+		(fields_autoplaced yes)
+		(property "Reference" "R6"
+			(at 195.58 25.4 0)
+			(show_name no)
+			(do_not_autoplace no)
+			(effects
+				(font
+					(size 1.27 1.27)
+				)
+			)
+		)
+		(property "Value" "ERA2AED753X"
+			(at 195.58 27.94 0)
+			(show_name no)
+			(do_not_autoplace no)
+			(effects
+				(font
+					(size 1.27 1.27)
+				)
+			)
+		)
+		(property "Footprint" "easyeda2kicad:R0402"
+			(at 195.58 39.37 0)
+			(hide yes)
+			(show_name no)
+			(do_not_autoplace no)
+			(effects
+				(font
+					(size 1.27 1.27)
+				)
+			)
+		)
+		(property "Datasheet" "https://lcsc.com/product-detail/New-Arrivals_PANASONIC-ERA2AED753X_C491105.html"
+			(at 195.58 41.91 0)
+			(hide yes)
+			(show_name no)
+			(do_not_autoplace no)
+			(effects
+				(font
+					(size 1.27 1.27)
+				)
+			)
+		)
+		(property "Description" "75k"
+			(at 195.58 31.75 0)
+			(show_name no)
+			(do_not_autoplace no)
+			(effects
+				(font
+					(size 1.27 1.27)
+				)
+			)
+		)
+		(property "Manufacturer" "PANASONIC(松下)"
+			(at 195.58 44.45 0)
+			(hide yes)
+			(show_name no)
+			(do_not_autoplace no)
+			(effects
+				(font
+					(size 1.27 1.27)
+				)
+			)
+		)
+		(property "MPN" "ERA2AED753X"
+			(at 195.58 46.99 0)
+			(hide yes)
+			(show_name no)
+			(do_not_autoplace no)
+			(effects
+				(font
+					(size 1.27 1.27)
+				)
+			)
+		)
+		(property "LCSC Part" "C491105"
+			(at 195.58 49.53 0)
+			(hide yes)
+			(show_name no)
+			(do_not_autoplace no)
+			(effects
+				(font
+					(size 1.27 1.27)
+				)
+			)
+		)
+		(pin "1"
+		)
+		(pin "2"
+		)
+		(instances
+			(project "right"
+				(path "/3171f1b4-f2dd-4471-8b63-415e18370dba"
+					(reference "R6")
+					(unit 1)
+				)
+			)
+		)
+	)
+	(symbol
 		(lib_id "PCM_SparkFun-PowerSymbol:GND")
 		(at 293.37 194.31 90)
@@
 	)
 	(symbol
-		(lib_id "easyeda2kicad:RT0402BRD0737K4L")
-		(at 195.58 31.75 0)
+		(lib_id "PCM_SparkFun-PowerSymbol:GND")
+		(at 260.35 241.3 270)
 		(unit 1)
 		(body_style 1)
@@
 		(dnp no)
 		(fields_autoplaced yes)
-		(property "Reference" "R15"
-			(at 195.58 26.162 0)
+		(property "Reference" "#PWR022"
+			(at 254 241.3 0)
+			(hide yes)
 			(show_name no)
 			(do_not_autoplace no)
@@
 			)
 		)
-		(property "Value" "RT0402BRD0737K4L"
-			(at 195.58 27.94 0)
-			(hide yes)
+		(property "Value" "GND"
+			(at 256.54 241.3 0)
 			(show_name no)
-			(do_not_autoplace no)
+			(do_not_autoplace yes)
 			(effects
 				(font
@@
 			)
 		)
-		(property "Footprint" ":R0402"
-			(at 195.58 39.37 0)
+		(property "Footprint" ""
+			(at 260.35 241.3 0)
 			(hide yes)
 			(show_name no)
@@
 		)
 		(property "Datasheet" ""
-			(at 195.58 31.75 0)
+			(at 260.35 241.3 0)
 			(hide yes)
 			(show_name no)
@@
 			)
 		)
-		(property "Description" "37k4"
-			(at 195.58 31.75 0)
-			(show_name no)
-			(do_not_autoplace no)
-			(effects
-				(font
-					(size 1.27 1.27)
-				)
-			)
-		)
-		(property "LCSC Part" "C852746"
-			(at 195.58 28.702 0)
+		(property "Description" "Power symbol creates a global label with name \"GND\" , ground"
+			(at 251.46 241.3 0)
+			(hide yes)
 			(show_name no)
 			(do_not_autoplace no)
@@
 		(pin "1"
 		)
-		(pin "2"
-		)
 		(instances
 			(project "right"
 				(path "/3171f1b4-f2dd-4471-8b63-415e18370dba"
-					(reference "R15")
+					(reference "#PWR022")
 					(unit 1)
 				)

Commit message: both sides done. changed few components for their basic or more affordable alternaatives.
Parts:
- removed C2: GRM155Z71A105KE01D, easyeda2kicad:C0402, symbol easyeda2kicad:GRM155Z71A105KE01D
- removed C4, C9: GRM033C71C104KE14D, easyeda2kicad:C0201, symbol easyeda2kicad:GRM033C71C104KE14D
- removed R12, R4, R7: RC0402FR-0710KL, easyeda2kicad:R0402, symbol easyeda2kicad:RC0402FR-0710KL
- removed R3: RC0402FR-07100KL, easyeda2kicad:R0402, symbol easyeda2kicad:RC0402FR-07100KL
- removed R5: RC0805FR-072M61L, easyeda2kicad:R0805, symbol easyeda2kicad:RC0805FR-072M61L
- removed U3: SN74LVC1G74DQER, :X2SON-8_L1.4-W1.0-P0.35-BL, symbol easyeda2kicad:SN74LVC1G74DQER
- added C10, C13: CL05B104KB54PNC, easyeda2kicad:C0402, symbol easyeda2kicad:GRM033C71C104KE14D
- added C9: CL05A105KA5NQNC, easyeda2kicad:C0402, symbol easyeda2kicad:GRM155Z71A105KE01D
- added R15, R18, R19: 0402WGF1002TCE, easyeda2kicad:R0402, symbol easyeda2kicad:RC0402FR-0710KL
- added R5: RC0402FR-07100KL, easyeda2kicad:R0402, symbol easyeda2kicad:RC0402FR-07100KL
- added R7: RTT022614FTH, easyeda2kicad:R0402, symbol easyeda2kicad:RC0805FR-072M61L
- added U10: SN74LVC1G74DQER, :X2SON-8_L1.4-W1.0-P0.35-BL, symbol easyeda2kicad:SN74LVC1G74DQER
- added U9: USBLC6-2SC6, Package_TO_SOT_SMD:SOT-23-6, symbol Power_Protection:USBLC6-2SC6
- C7, C8: value GRM155C71C105KE11D -> CL05A105KA5NQNC; LCSC Part C576449 -> C52923
- R10, R14, R16, R9: value RC0402FR-075K1L -> 0402WGF5101TCE; LCSC Part C105872 -> C25905
- R11: value RC0201FR-07680RL -> RC0402FR-07680RL; footprint easyeda2kicad:R0201 -> easyeda2kicad:R0402; LCSC Part C274876 -> C137948
- R13: value RC0402FR-0710KL -> 0402WGF1002TCE; LCSC Part C60490 -> C25744
- R17: value RC0402FR-071ML -> 0402WGF1004TCE; LCSC Part C138033 -> C26083
Connections:
- net BAT+: now also C10.1, R19.2, U10.7 (~{PRE}), U10.8 (VCC)
- net BAT_ALTR: now also R13.1
- net CHRG: now also R15.1
- net D+: now also U9.1 (I/O1), U9.6 (I/O1)
- net D-: now also U9.3 (I/O2), U9.4 (I/O2)
- net GND: now also C10.2, C13.1, C9.2, R5.2, U10.4 (GND), U9.2 (GND)
- net PMOS_gate: now also U10.2 (D), U10.3 (~{Q})
- net PWR_BTN: now also R5.1, R7.1
- net STDBY: now also R18.1; no longer R13.1
- net VDD_nRF: now also R15.2, R18.2
- net at D1.2, U1.2 (A): now also C9.1, R7.2
- net VBUS_RAW: now reaches F1.1, USBC1.A4B9 (VBUS), USBC1.B4A9 (VBUS)
- net VBUS_RAW: now also U9.5 (VBUS)
- net at U1.4 (Y): now also U10.1 (CLK)
- new net: C13.2, R19.1, U10.6 (~{CLR})
- no-connect marks 20 -> 21

Commit message: first panelization... changing parts because of availability
Parts:
- removed R5: RC0402FR-07100KL, easyeda2kicad:R0402, symbol easyeda2kicad:RC0402FR-07100KL
- added R5: 0402WGF1002TCE, easyeda2kicad:R0402, symbol easyeda2kicad:RC0402FR-0710KL
- C6: value GRM033C71C104KE14D -> CL05B104KB54PNC; footprint easyeda2kicad:C0201 -> easyeda2kicad:C0402; LCSC Part C85923 -> C307331
- R1: value RC0402FR-071ML -> 0402WGF1004TCE; LCSC Part C138033 -> C26083
- R8: value RC0402FR-0710KL -> 0402WGF1002TCE; LCSC Part C60490 -> C25744
Connections:
- net GND: now also R5.2
- net PWR_BTN: now also R5.1
- net PWR_BTN_PRESS: now also U2.4 (AI4); no longer U2.30 (P17)

Commit message: added lcsc part # for USBLC6-2SC6
Parts:
- U9: LSCS Part (none) -> C7519
Changed lines of the file:
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@@
+			)
+		)
+		(property "LSCS Part" "C7519"
+			(at 280.67 214.63 0)
+			(hide yes)
+			(show_name no)
+			(do_not_autoplace no)
+			(effects
+				(font
+					(size 1.27 1.27)
+				)
 			)
 		)
